Commit message: base floating and affected by gravity

File: src/space_robot/description/gazebo/depth_camera.gazebo.xacro (robot description, xacro)
@@ -19,8 +19,4 @@
                 <visualize>true</visualize>
                 <topic>rgbd_camera</topic>
-                <plugin
-                    filename="RosGzPointCloud"
-                    name="ros_gz_point_cloud::PointCloud">
-                </plugin>
             </sensor>
             <!-- <sensor name="rgbd_camera" type="rgbd_camera">

File: src/space_robot/description/urdf/robot_model/robot_base.urdf.xacro (robot description, xacro)
@@ -2,9 +2,4 @@
 <robot xmlns:xacro="http://www.ros.org/wiki/xacro" name="robot_base">
     <xacro:macro name="base" params="name cubic_size base_mass base_inertia material parent_link *origin">
-        <joint name="base_joint" type="floating">
-            <parent link="${parent_link}"/>
-            <child link="${name}_link"/>
-            <xacro:insert_block name="origin"/>
-        </joint>
         <link name="${name}_link">
             <visual>

File: src/space_robot/description/urdf/space_robot.urdf.xacro (robot description, xacro)
@@ -3,5 +3,4 @@
     <xacro:arg name="prefix" default="" />
     <xacro:arg name="use_gazebo" default="true" />
-    <link name="world"/>
     <xacro:include filename="$(find space_robot)/description/urdf/robot_description.urdf.xacro"/>
     <xacro:srobot parent="world" prefix="{arg prefix}">
