Commit message: reconstruct and moveit work with gazebo without connection controllers

File: src/space_robot_learning/description/gazebo/robot.gazebo.xacro (robot description, xacro)
@@ -1,9 +1,9 @@
 <?xml version="1.0"?>
 <robot xmlns:xacro="http://ros.org/wiki/xacro">
-  <xacro:macro name="srobot_gazebo">
+  <xacro:macro name="srobot_gazebo" params="prefix">
     <!-- gz_ros_control plugin -->
     <gazebo>
       <plugin filename="gz_ros2_control-system" name="gz_ros2_control::GazeboSimROS2ControlPlugin">
-        <parameters>$(find space_robot)/config/controllers.yaml</parameters>
+        <parameters>$(find space_robot_learning)/bringup/config/controllers.yaml</parameters>
       </plugin>
       <plugin filename="gz-sim-pose-publisher-system" name="gz::sim::systems::PosePublisher">
@@ -15,5 +15,5 @@
     </gazebo>
     <!-- Base -->
-    <gazebo reference="base_link">
+    <gazebo reference="${prefix}base_link">
       <material>
         <script>
@@ -24,5 +24,5 @@
     </gazebo>
     <!-- Link1 -->
-    <gazebo reference="link_1">
+    <gazebo reference="${prefix}link_1">
       <mu1>0.2</mu1>
       <mu2>0.2</mu2>
@@ -35,5 +35,5 @@
     </gazebo>
     <!-- Link2 -->
-    <gazebo reference="link_2">
+    <gazebo reference="${prefix}link_2">
       <mu1>0.2</mu1>
       <mu2>0.2</mu2>

File: src/space_robot_learning/description/urdf/robot_description.urdf.xacro (robot description, xacro)
@@ -1,14 +1,6 @@
 <?xml version="1.0"?>
 <robot xmlns:xacro="http://www.ros.org/wiki/xacro">
-    <xacro:macro name="srobot" params="parent use_gazebo *origin">
+    <xacro:macro name="srobot" params="parent prefix *origin">
         <xacro:property name="axel_offset" value="0.005"/>
-        <xacro:unless value="${use_gazebo}">
-            <link name="${parent}"/>
-            <joint name="base_joint" type="floating">
-                <origin xyz="0 0 0" rpy="0 0 0"/>
-                <parent link="${parent}" />
-                <child link="base_link" />
-            </joint>
-        </xacro:unless>
         <!-- robot base -->
         <xacro:property name="base_size" value="1.4" />  <!-- Unit: m -->
@@ -16,5 +8,5 @@
         <xacro:property name="base_inertia" value="50" />    <!-- Unit: kg*m^2 -->
         <xacro:property name="base_material" value="brown"/>
-        <xacro:include filename="$(find space_robot)/description/urdf/robot_model/robot_base.urdf.xacro"/>
+        <xacro:include filename="$(find space_robot_learning)/description/urdf/robot_model/robot_base.urdf.xacro"/>
         <xacro:base
             name="base"
@@ -33,5 +25,5 @@
         <xacro:property name="link_1_inertia" value="7.8408"/>
         <xacro:property name="link_1_material" value="yellow"/>
-        <xacro:include filename="$(find space_robot)/description/urdf/robot_model/robot_link.urdf.xacro"/>
+        <xacro:include filename="$(find space_robot_learning)/description/urdf/robot_model/robot_link.urdf.xacro"/>
         <xacro:link
             name="link_1"
@@ -53,5 +45,5 @@
         <xacro:property name="link_2_inertia" value="7.8408"/>
         <xacro:property name="link_2_material" value="grey"/>
-        <xacro:include filename="$(find space_robot)/description/urdf/robot_model/robot_link.urdf.xacro"/>
+        <xacro:include filename="$(find space_robot_learning)/description/urdf/robot_model/robot_link.urdf.xacro"/>
         <xacro:link
             name="link_2"
@@ -66,9 +58,9 @@
             <origin xyz="${0.5 * axel_offset + link_1_length} 0 0" rpy="0 0 0"/>
         </xacro:link>
-        <xacro:include filename="$(find space_robot)/description/urdf/depth_camera.urdf.xacro"/>
+        <xacro:include filename="$(find space_robot_learning)/description/urdf/depth_camera.urdf.xacro"/>
         <xacro:depth_camera parent_link="link_2" camera_name="front_depth_cam">
             <origin xyz="${link_2_length} ${link_2_radius + 0.001} 0" rpy="0 0 0"/>
         </xacro:depth_camera>
-        <xacro:include filename="$(find space_robot)/description/gazebo/depth_camera.gazebo.xacro"/>
+        <xacro:include filename="$(find space_robot_learning)/description/gazebo/depth_camera.gazebo.xacro"/>
         <xacro:depth_camera_gazebo camera_name="front_depth_cam"/>
     </xacro:macro>
