Commit message: fix planning issue_2

File: src/space_robot_config/config/space_robot.urdf.xacro (robot description, xacro)
@@ -12,3 +12,10 @@
     <xacro:include filename="$(find space_robot_config)/description/ros2_control/space_robot.ros2_control.xacro" />
     <xacro:space_robot_ros2_control name="FakeSystem" initial_positions_file="$(arg initial_positions_file)"/>
+    <!-- Gazebo -->
+    <xacro:if value="$(arg use_gazebo)">
+        <xacro:include filename="$(find space_robot_config)/description/gazebo/depth_camera.gazebo.xacro"/>
+        <xacro:depth_camera_gazebo camera_name="front_depth_cam"/>
+        <xacro:include filename="$(find space_robot_config)/description/gazebo/robot.gazebo.xacro" />
+        <xacro:srobot_gazebo name="srobot_gazebo"/>
+    </xacro:if>
 </robot>

File: src/space_robot_config/description/gazebo/robot.gazebo.xacro (robot description, xacro)
@@ -1,5 +1,5 @@
 <?xml version="1.0"?>
 <robot xmlns:xacro="http://ros.org/wiki/xacro">
-  <xacro:macro name="srobot_gazebo">
+    <xacro:macro name="srobot_gazebo" params="name">
     <!-- gz_ros_control plugin -->
     <gazebo>
@@ -13,4 +13,11 @@
           <update_frequency>10</update_frequency>
       </plugin>
+    </gazebo>
+    <gazebo>
+      <joint name='base_joint' type='fixed'>
+        <pose relative_to='__model__'>0 0 0 0 0 0</pose>
+        <parent>world</parent>
+        <child>base_link</child>
+      </joint>
     </gazebo>
     <!-- Base -->
@@ -45,4 +52,4 @@
       </material>
     </gazebo>
-  </xacro:macro>
+    </xacro:macro>
 </robot>

File: src/space_robot_config/description/urdf/robot_description.urdf.xacro (robot description, xacro)
@@ -3,12 +3,10 @@
     <xacro:macro name="srobot" params="parent use_gazebo *origin">
         <xacro:property name="axel_offset" value="0.005"/>
-        <xacro:unless value="${use_gazebo}">
-            <link name="${parent}"/>
-            <joint name="base_joint" type="floating">
-                <origin xyz="0 0 0" rpy="0 0 0"/>
-                <parent link="${parent}" />
-                <child link="base_link" />
-            </joint>
-        </xacro:unless>
+        <link name="${parent}"/>
+        <joint name="base_joint" type="floating">
+            <origin xyz="0 0 0" rpy="0 0 0"/>
+            <parent link="${parent}" />
+            <child link="base_link" />
+        </joint>
         <!-- robot base -->
         <xacro:property name="base_size" value="1.4" />  <!-- Unit: m -->
@@ -70,6 +68,4 @@
             <origin xyz="${link_2_length} ${link_2_radius + 0.001} 0" rpy="0 0 0"/>
         </xacro:depth_camera>
-        <xacro:include filename="$(find space_robot_config)/description/gazebo/depth_camera.gazebo.xacro"/>
-        <xacro:depth_camera_gazebo camera_name="front_depth_cam"/>
     </xacro:macro>
 </robot>

Commit message: solve moveit_gazebo problem 8

File: src/space_robot_config/config/space_robot.urdf.xacro (robot description, xacro)
@@ -2,5 +2,5 @@
 <robot xmlns:xacro="http://www.ros.org/wiki/xacro" name="space_robot">
     <xacro:arg name="initial_positions_file" default="initial_positions.yaml" />
-    <xacro:arg name="use_gazebo" default="true" />
+    <xacro:arg name="use_gazebo" default="false" />
     <!-- Import space_robot urdf file -->
     <xacro:include filename="$(find space_robot_config)/description/urdf/robot_description.urdf.xacro"/>
@@ -11,5 +11,6 @@
     <!-- Import control_xacro -->
     <xacro:include filename="$(find space_robot_config)/description/ros2_control/space_robot.ros2_control.xacro" />
-    <xacro:space_robot_ros2_control name="FakeSystem" initial_positions_file="$(arg initial_positions_file)"/>
+    <xacro:space_robot_ros2_control name="FakeSystem" initial_positions_file="$(arg initial_positions_file)"
+        use_gazebo="$(arg use_gazebo)"/>
     <!-- Gazebo -->
     <xacro:if value="$(arg use_gazebo)">

File: src/space_robot_config/description/ros2_control/space_robot.ros2_control.xacro (robot description, xacro)
@@ -1,10 +1,15 @@
 <?xml version="1.0"?>
 <robot xmlns:xacro="http://www.ros.org/wiki/xacro">
-    <xacro:macro name="space_robot_ros2_control" params="name initial_positions_file">
+    <xacro:macro name="space_robot_ros2_control" params="name initial_positions_file use_gazebo">
         <xacro:property name="initial_positions" value="${xacro.load_yaml(initial_positions_file)['initial_positions']}"/>
         <ros2_control name="${name}" type="system">
             <hardware>
                 <!-- By default, set up controllers for simulation. This won't work on real hardware -->
-                <plugin>mock_components/GenericSystem</plugin>
+                <xacro:if value="${use_gazebo}">
+                    <plugin>gz_ros2_control/GazeboSimSystem</plugin>
+                </xacro:if>
+                <xacro:unless value='${use_gazebo}'>
+                    <plugin>mock_components/GenericSystem</plugin>
+                </xacro:unless>
             </hardware>
             <joint name="link_1_joint">
