Commit message: solve moveit_gazebo problem 9

File: src/space_robot_config/description/gazebo/robot.gazebo.xacro (robot description, xacro)
@@ -13,11 +13,4 @@
         <joint_name>link_2_joint</joint_name>
       </plugin>
-    </gazebo>
-    <gazebo>
-      <joint name='base_joint' type='fixed'>
-        <pose relative_to='__model__'>0 0 0 0 0 0</pose>
-        <parent>world</parent>
-        <child>base_link</child>
-      </joint>
     </gazebo>
     <!-- Base -->

File: src/space_robot_config/description/urdf/robot_description.urdf.xacro (robot description, xacro)
@@ -3,10 +3,12 @@
     <xacro:macro name="srobot" params="parent use_gazebo *origin">
         <xacro:property name="axel_offset" value="0.005"/>
-        <link name="${parent}"/>
-        <joint name="base_joint" type="floating">
-            <origin xyz="0 0 0" rpy="0 0 0"/>
-            <parent link="${parent}" />
-            <child link="base_link" />
-        </joint>
+        <xacro:unless value="${use_gazebo}">
+            <link name="${parent}"/>
+            <joint name="base_joint" type="floating">
+                <origin xyz="0 0 0" rpy="0 0 0"/>
+                <parent link="${parent}" />
+                <child link="base_link" />
+            </joint>
+        </xacro:unless>
         <!-- robot base -->
         <xacro:property name="base_size" value="1.4" />  <!-- Unit: m -->

Commit message: backup

File: src/space_robot_config/description/gazebo/robot.gazebo.xacro (robot description, xacro)
@@ -13,4 +13,10 @@
         <joint_name>link_2_joint</joint_name>
       </plugin>
+    </gazebo>
+    <gazebo reference="left_finger_joint">
+        <preserveFixedJoint>false</preserveFixedJoint>
+    </gazebo>
+    <gazebo reference="right_finger_joint">
+        <preserveFixedJoint>false</preserveFixedJoint>
     </gazebo>
     <!-- Base -->

File: src/space_robot_config/description/urdf/robot_description.urdf.xacro (robot description, xacro)
@@ -66,4 +66,11 @@
             <origin xyz="${0.5 * axel_offset + link_1_length} 0 0" rpy="0 0 0"/>
         </xacro:link>
+        <!-- gripper -->
+        <xacro:include filename="$(find space_robot_config)/description/urdf/robot_model/gripper.urdf.xacro" />
+        <xacro:gripper_base parent="link_2">
+            <origin xyz="${link_2_length + 0.01} 0 0" rpy="${0.5 * pi} 0 0" />
+        </xacro:gripper_base>
+        <xacro:finger prefix="left" reflect="-" />
+        <xacro:finger prefix="right" reflect="" />
         <xacro:include filename="$(find space_robot_config)/description/urdf/depth_camera.urdf.xacro"/>
         <xacro:depth_camera parent_link="link_2" camera_name="front_depth_cam">

File: src/tmp_space_robot_config_with_gripper/config/space_robot.ros2_control.xacro (robot description, xacro)
@@ -1,15 +1,10 @@
 <?xml version="1.0"?>
 <robot xmlns:xacro="http://www.ros.org/wiki/xacro">
-    <xacro:macro name="space_robot_ros2_control" params="name initial_positions_file use_gazebo">
-        <xacro:property name="initial_positions" value="${xacro.load_yaml(initial_positions_file)['initial_positions']}"/>
+    <xacro:macro name="space_robot_ros2_control" params="name initial_positions_file">
+        <xacro:property name="initial_positions" value="${load_yaml(initial_positions_file)['initial_positions']}"/>
         <ros2_control name="${name}" type="system">
             <hardware>
                 <!-- By default, set up controllers for simulation. This won't work on real hardware -->
-                <xacro:if value="${use_gazebo}">
-                    <plugin>gz_ros2_control/GazeboSimSystem</plugin>
-                </xacro:if>
-                <xacro:unless value='${use_gazebo}'>
-                    <plugin>mock_components/GenericSystem</plugin>
-                </xacro:unless>
+                <plugin>mock_components/GenericSystem</plugin>
             </hardware>
             <joint name="link_1_joint">
